File: schematic/colecovision_controller.kicad_pcb (KiCad board)
At the start: 2 copper layers, 112.4 x 59.1 mm, 56 parts, among them J1 Conn_01x09, SW1 SW_AST, SW10 SW_9, SW11 SW_6, SW12 SW_3, SW13 SW_LEFT, SW14 SW_UP, SW15 SW_DOWN, SW16 SW_RIGHT, SW17 SW_ARM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

Commit message: update to kicad 6, mit license added
Other:
- net class Default removed
- net class keypad removed
