File: schematic/colecovision_controller.kicad_sch (KiCad schematic)
At the start: 56 parts, among them J1 Conn_01x09, SW1 SW_AST, SW10 SW_9, SW11 SW_6, SW12 SW_3, SW13 SW_LEFT, SW14 SW_UP, SW15 SW_DOWN, SW16 SW_RIGHT, SW17 SW_ARM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

Commit message: updated to fix arm/fire button position. Now matches original controller.
Parts:
- renumbered D28 to D27, D27 to D28, SW18 to SW17, SW17 to SW18
Changed lines of the file:
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@@
   (symbol (lib_id "Switch:SW_MEC_5E") (at 85.09 71.12 180) (unit 1)
     (in_bom yes) (on_board yes) (dnp no)
-    (property "Reference" "SW18" (at 85.09 79.375 0)
+    (property "Reference" "SW17" (at 85.09 79.375 0)
       (effects (font (size 1.27 1.27)))
     )
@@
       (project "colecovision_controller"
         (path "/909efb56-6ead-4c33-b43f-ae05a3878582"
+          (reference "SW17") (unit 1)
+        )
+      )
+    )
+  )
+  (symbol (lib_id "Switch:SW_MEC_5E") (at 85.09 85.09 180) (unit 1)
+    (in_bom yes) (on_board yes) (dnp no)
+    (property "Reference" "SW18" (at 85.09 93.345 0)
+      (effects (font (size 1.27 1.27)))
+    )
+    (property "Value" "SW_ARM" (at 85.09 95.25 0)
+      (effects (font (size 1.27 1.27)))
+    )
+    (property "Footprint" "Button_Switch_THT:SW_TH_Tactile_Omron_B3F-10xx" (at 85.09 85.09 0)
+      (effects (font (size 1.27 1.27)) hide)
+    )
+    (property "Datasheet" "~" (at 85.09 85.09 0)
+      (effects (font (size 1.27 1.27)) hide)
+    )
+    (pin "1")
+    (pin "2")
+    (pin "3")
+    (pin "4")
+    (instances
+      (project "colecovision_controller"
+        (path "/909efb56-6ead-4c33-b43f-ae05a3878582"
           (reference "SW18") (unit 1)
-        )
-      )
-    )
-  )
-  (symbol (lib_id "Switch:SW_MEC_5E") (at 85.09 85.09 180) (unit 1)
-    (in_bom yes) (on_board yes) (dnp no)
-    (property "Reference" "SW17" (at 85.09 93.345 0)
-      (effects (font (size 1.27 1.27)))
-    )
-    (property "Value" "SW_ARM" (at 85.09 95.25 0)
-      (effects (font (size 1.27 1.27)))
-    )
-    (property "Footprint" "Button_Switch_THT:SW_TH_Tactile_Omron_B3F-10xx" (at 85.09 85.09 0)
-      (effects (font (size 1.27 1.27)) hide)
-    )
-    (property "Datasheet" "~" (at 85.09 85.09 0)
-      (effects (font (size 1.27 1.27)) hide)
-    )
-    (pin "1")
-    (pin "2")
-    (pin "3")
-    (pin "4")
-    (instances
-      (project "colecovision_controller"
-        (path "/909efb56-6ead-4c33-b43f-ae05a3878582"
-          (reference "SW17") (unit 1)
         )
       )
@@
   (symbol (lib_id "Device:D_Small") (at 74.93 85.09 180) (unit 1)
     (in_bom yes) (on_board yes) (dnp no)
-    (property "Reference" "D27" (at 74.93 90.3478 0)
+    (property "Reference" "D28" (at 74.93 90.3478 0)
       (effects (font (size 1.27 1.27)))
     )
@@
       (project "colecovision_controller"
         (path "/909efb56-6ead-4c33-b43f-ae05a3878582"
+          (reference "D28") (unit 1)
+        )
+      )
+    )
+  )
+  (symbol (lib_id "Device:D_Small") (at 74.93 73.66 180) (unit 1)
+    (in_bom yes) (on_board yes) (dnp no)
+    (property "Reference" "D27" (at 74.93 78.9178 0)
+      (effects (font (size 1.27 1.27)))
+    )
+    (property "Value" "D_Small" (at 74.93 76.6064 0)
+      (effects (font (size 1.27 1.27)))
+    )
+    (property "Footprint" "Diode_THT:D_DO-35_SOD27_P7.62mm_Horizontal" (at 74.93 73.66 90)
+      (effects (font (size 1.27 1.27)) hide)
+    )
+    (property "Datasheet" "~" (at 74.93 73.66 90)
+      (effects (font (size 1.27 1.27)) hide)
+    )
+    (pin "1")
+    (pin "2")
+    (instances
+      (project "colecovision_controller"
+        (path "/909efb56-6ead-4c33-b43f-ae05a3878582"
           (reference "D27") (unit 1)
         )
       )
-    )
-  )
-  (symbol (lib_id "Device:D_Small") (at 74.93 73.66 180) (unit 1)
-    (in_bom yes) (on_board yes) (dnp no)
-    (property "Reference" "D28" (at 74.93 78.9178 0)
-      (effects (font (size 1.27 1.27)))
-    )
-    (property "Value" "D_Small" (at 74.93 76.6064 0)
-      (effects (font (size 1.27 1.27)))
-    )
-    (property "Footprint" "Diode_THT:D_DO-35_SOD27_P7.62mm_Horizontal" (at 74.93 73.66 90)
-      (effects (font (size 1.27 1.27)) hide)
-    )
-    (property "Datasheet" "~" (at 74.93 73.66 90)
-      (effects (font (size 1.27 1.27)) hide)
-    )
-    (pin "1")
-    (pin "2")
-    (instances
-      (project "colecovision_controller"
-        (path "/909efb56-6ead-4c33-b43f-ae05a3878582"
-          (reference "D28") (unit 1)
-        )
-      )
